File: pcb.kicad_sch (KiCad schematic)
At the start: 26 parts, among them J1 USB3_B_Micro, J2 Conn_01x04_Pin, J3 Conn_01x04_Pin, J4 Conn_01x04_Pin, SW1 SW_SPDT, U1 STM32F103C8Tx, U2 AMS1117-3.3, Y1 16Mhz

Commit message: first commit
Parts:
- removed J1: USB3_B_Micro, Package_DFN_QFN:WDFN-10-1EP_3x3mm_P0.5mm_EP1.8x2.5mm, symbol Connector:USB3_B_Micro
- added H1, H2, H3, H4: MountingHole, MountingHole:MountingHole_2.5mm, symbol Mechanical:MountingHole
- added J5: USB_B_Micro, Package_DFN_QFN:WDFN-10-1EP_3x3mm_P0.5mm_EP1.8x2.5mm, symbol Connector:USB_B_Micro
Connections:
- net GND is gone; now on net +3.3V: C1.2, C10.2, C11.2, C12.2, C13.2, C2.2, C3.2, C4.2, C5.2, C6.2, C7.2, C8.2, C9.2, J2.4 (Pin_4), J3.4 (Pin_4), J4.4 (Pin_4), R3.2, SW1.1 (A), U1.23 (VSS), U1.35 (VSS), U1.47 (VSS), U1.8 (VSSA), U2.1 (GND)
- net hse in is gone; now on net +3.3V: C10.1, U1.5 (PD0), Y1.1, Y1.2 (G), Y1.4 (G)
- net +3.3V: now also J5.5 (GND)
- net VBUS: now also J5.1 (VBUS)
- net usb d+: now also J5.3 (D+)
- net usb d-: now also J5.2 (D-)
- no-connect marks 34 -> 29
Other:
- note added: "mounting holes"
- moved on the sheet: SW1

Commit message: Add STM32 KiCad PCB design
Connections:
- net +3.3V: no longer C1.2, C10.1, C10.2, C11.2, C12.2, C13.2, C2.2, C3.2, C4.2, C5.2, C6.2, C7.2, C8.2, C9.2, J2.4 (Pin_4), J3.4 (Pin_4), J4.4 (Pin_4), J5.5 (GND), R3.2, SW1.1 (A), U1.23 (VSS), U1.35 (VSS), U1.47 (VSS), U1.5 (PD0), U1.8 (VSSA), U2.1 (GND), Y1.1, Y1.2 (G), Y1.4 (G)
- new net GND: C1.2, C10.2, C11.2, C12.2, C13.2, C2.2, C3.2, C4.2, C5.2, C6.2, C7.2, C8.2, C9.2, J2.4 (Pin_4), J3.4 (Pin_4), J4.4 (Pin_4), J5.5 (GND), R3.2, SW1.1 (A), U1.23 (VSS), U1.35 (VSS), U1.47 (VSS), U1.8 (VSSA), U2.1 (GND), Y1.2 (G), Y1.4 (G)
- new net hse in: C10.1, U1.5 (PD0), Y1.1
Changed lines of the file:
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@@
 	)
 	(junction
-		(at 130.81 60.96)
-		(diameter 0)
-		(color 0 0 0 0)
-	)
-	(junction
 		(at 146.05 80.01)
 		(diameter 0)
@@
 	)
 	(junction
-		(at 110.49 38.1)
-		(diameter 0)
-		(color 0 0 0 0)
-	)
-	(junction
 		(at 175.26 39.37)
 		(diameter 0)
@@
 	)
 	(junction
-		(at 67.31 41.91)
+		(at 110.49 38.1)
 		(diameter 0)
 		(color 0 0 0 0)
@@
 	)
 	(junction
-		(at 137.16 60.96)
+		(at 153.67 60.96)
 		(diameter 0)
 		(color 0 0 0 0)
@@
 	(wire
 		(pts
-			(xy 182.88 24.13) (xy 182.88 29.21)
+			(xy 153.67 60.96) (xy 160.02 60.96)
 		)
 		(stroke
@@
 	(wire
 		(pts
-			(xy 67.31 44.45) (xy 59.69 44.45)
+			(xy 182.88 24.13) (xy 182.88 29.21)
 		)
 		(stroke
@@
 	(wire
 		(pts
+			(xy 233.68 76.2) (xy 233.68 80.01)
+		)
+		(stroke
+			(width 0)
+			(type default)
+		)
+	)
+	(wire
+		(pts
 			(xy 251.46 29.21) (xy 259.08 29.21)
 		)
@@
 	(wire
 		(pts
-			(xy 228.6 93.98) (xy 233.68 93.98)
+			(xy 153.67 58.42) (xy 153.67 60.96)
 		)
 		(stroke
@@
 	(wire
 		(pts
-			(xy 182.88 29.21) (xy 205.74 29.21)
+			(xy 152.4 62.23) (xy 160.02 62.23)
 		)
 		(stroke
@@
 	(wire
 		(pts
-			(xy 212.09 82.55) (xy 212.09 109.22)
+			(xy 182.88 29.21) (xy 205.74 29.21)
 		)
 		(stroke
@@
 	(wire
 		(pts
-			(xy 110.49 30.48) (xy 119.38 30.48)
+			(xy 212.09 82.55) (xy 212.09 109.22)
 		)
 		(stroke
@@
 	(wire
 		(pts
-			(xy 245.11 95.25) (xy 245.11 105.41)
+			(xy 110.49 30.48) (xy 119.38 30.48)
 		)
 		(stroke
@@
 	(wire
 		(pts
+			(xy 149.86 60.96) (xy 149.86 68.58)
+		)
+		(stroke
+			(width 0)
+			(type default)
+		)
+	)
+	(wire
+		(pts
 			(xy 180.34 125.73) (xy 177.8 125.73)
 		)
@@
 	(wire
 		(pts
+			(xy 149.86 68.58) (xy 124.46 68.58)
+		)
+		(stroke
+			(width 0)
+			(type default)
+		)
+	)
+	(wire
+		(pts
 			(xy 154.94 95.25) (xy 160.02 95.25)
 		)
@@
 	(wire
 		(pts
+			(xy 124.46 68.58) (xy 124.46 60.96)
+		)
+		(stroke
+			(width 0)
+			(type default)
+		)
+	)
+	(wire
+		(pts
 			(xy 137.16 123.19) (xy 143.51 123.19)
 		)
@@
 	(wire
 		(pts
+			(xy 59.69 44.45) (xy 63.5 44.45)
+		)
+		(stroke
+			(width 0)
+			(type default)
+		)
+	)
+	(wire
+		(pts
 			(xy 167.64 39.37) (xy 172.72 39.37)
 		)
@@
 	(wire
 		(pts
-			(xy 146.05 80.01) (xy 151.13 80.01)
+			(xy 146.05 80.01) (xy 152.4 80.01)
 		)
 		(stroke
@@
 	(wire
 		(pts
+			(xy 245.11 96.52) (xy 245.11 95.25)
+		)
+		(stroke
+			(width 0)
+			(type default)
+		)
+	)
+	(wire
+		(pts
 			(xy 213.36 114.3) (xy 213.36 119.38)
 		)
@@
 	(wire
 		(pts
-			(xy 137.16 60.96) (xy 160.02 60.96)
+			(xy 63.5 40.64) (xy 67.31 40.64)
 		)
 		(stroke
@@
 	(wire
 		(pts
+			(xy 63.5 44.45) (xy 63.5 40.64)
+		)
+		(stroke
+			(width 0)
+			(type default)
+		)
+	)
+	(wire
+		(pts
 			(xy 229.87 88.9) (xy 237.49 88.9)
 		)
@@
 	(wire
 		(pts
-			(xy 137.16 118.11) (xy 154.94 118.11)
+			(xy 152.4 62.23) (xy 152.4 80.01)
 		)
 		(stroke
@@
 	(wire
 		(pts
-			(xy 30.48 57.15) (xy 52.07 57.15)
+			(xy 137.16 118.11) (xy 154.94 118.11)
 		)
 		(stroke
@@
 	(wire
 		(pts
-			(xy 233.68 93.98) (xy 233.68 80.01)
+			(xy 30.48 57.15) (xy 52.07 57.15)
 		)
 		(stroke
@@
 	(wire
 		(pts
-			(xy 119.38 60.96) (xy 130.81 60.96)
+			(xy 124.46 60.96) (xy 119.38 60.96)
 		)
 		(stroke
@@
 	(wire
 		(pts
-			(xy 151.13 80.01) (xy 151.13 62.23)
+			(xy 149.86 60.96) (xy 153.67 60.96)
 		)
 		(stroke
@@
 	(wire
 		(pts
-			(xy 130.81 60.96) (xy 137.16 60.96)
-		)
-		(stroke
-			(width 0)
-			(type default)
-		)
-	)
-	(wire
-		(pts
 			(xy 228.6 36.83) (xy 228.6 40.64)
 		)
@@
 	(wire
 		(pts
-			(xy 110.49 38.1) (xy 110.49 41.91)
-		)
-		(stroke
-			(width 0)
-			(type default)
-		)
-	)
-	(wire
-		(pts
-			(xy 151.13 62.23) (xy 160.02 62.23)
-		)
-		(stroke
-			(width 0)
-			(type default)
-		)
-	)
-	(wire
-		(pts
 			(xy 156.21 54.61) (xy 160.02 54.61)
 		)
@@
 	(wire
 		(pts
-			(xy 67.31 41.91) (xy 67.31 44.45)
-		)
-		(stroke
-			(width 0)
-			(type default)
-		)
-	)
-	(wire
-		(pts
 			(xy 110.49 123.19) (xy 121.92 123.19)
 		)
@@
 	)
 	(label "hse out"
-		(at 151.13 62.23 0)
+		(at 152.4 64.77 0)
 		(effects
 			(font
@@
 	)
 	(label "hse in"
-		(at 153.67 60.96 0)
+		(at 153.67 58.42 0)
 		(effects
 			(font
@@
 	(symbol
 		(lib_id "power:VBUS")
-		(at 228.6 93.98 0)
+		(at 233.68 76.2 0)
 		(unit 1)
 		(body_style 1)
@@
 		(fields_autoplaced yes)
 		(property "Reference" "#PWR013"
-			(at 228.6 97.79 0)
+			(at 233.68 80.01 0)
 			(hide yes)
 			(show_name no)
@@
 		)
 		(property "Value" "VBUS"
-			(at 228.6 88.9 0)
+			(at 233.68 71.12 0)
 			(show_name no)
 			(do_not_autoplace no)
@@
 		)
 		(property "Footprint" "Package_QFP:TQFP-44_10x10mm_P0.8mm"
-			(at 228.6 93.98 0)
+			(at 233.68 76.2 0)
 			(hide yes)
 			(show_name no)
@@
 		)
 		(property "Datasheet" ""
-			(at 228.6 93.98 0)
+			(at 233.68 76.2 0)
 			(hide yes)
 			(show_name no)
@@
 		)
 		(property "Description" "Power symbol creates a global label with name \"VBUS\""
-			(at 228.6 93.98 0)
+			(at 233.68 76.2 0)
 			(hide yes)
 			(show_name no)
@@
 	(symbol
 		(lib_id "power:GND")
-		(at 110.49 41.91 0)
+		(at 110.49 38.1 0)
 		(unit 1)
 		(body_style 1)
@@
 		(fields_autoplaced yes)
 		(property "Reference" "#PWR03"
-			(at 110.49 48.26 0)
+			(at 110.49 44.45 0)
 			(hide yes)
 			(show_name no)
@@
 		)
 		(property "Value" "GND"
-			(at 110.49 46.99 0)
+			(at 110.49 43.18 0)
 			(show_name no)
 			(do_not_autoplace no)
@@
 		)
 		(property "Footprint" ""
-			(at 110.49 41.91 0)
+			(at 110.49 38.1 0)
 			(hide yes)
 			(show_name no)
@@
 		)
 		(property "Datasheet" ""
-			(at 110.49 41.91 0)
+			(at 110.49 38.1 0)
 			(hide yes)
 			(show_name no)
@@
 		)
 		(property "Description" "Power symbol creates a global label with name \"GND\" , ground"
-			(at 110.49 41.91 0)
+			(at 110.49 38.1 0)
 			(hide yes)
 			(show_name no)
@@
 	(symbol
 		(lib_id "power:GND")
-		(at 245.11 105.41 0)
+		(at 245.11 96.52 0)
 		(mirror y)
 		(unit 1)
@@
 		(fields_autoplaced yes)
 		(property "Reference" "#PWR012"
-			(at 245.11 111.76 0)
+			(at 245.11 102.87 0)
 			(hide yes)
 			(show_name no)
@@
 		)
 		(property "Value" "GND"
-			(at 245.11 110.49 0)
+			(at 245.11 101.6 0)
 			(show_name no)
 			(do_not_autoplace no)
@@
 		)
 		(property "Footprint" ""
-			(at 245.11 105.41 0)
+			(at 245.11 96.52 0)
 			(hide yes)
 			(show_name no)
@@
 		)
 		(property "Datasheet" ""
-			(at 245.11 105.41 0)
+			(at 245.11 96.52 0)
 			(hide yes)
 			(show_name no)
@@
 		)
 		(property "Description" "Power symbol creates a global label with name \"GND\" , ground"
-			(at 245.11 105.41 0)
+			(at 245.11 96.52 0)
 			(hide yes)
 			(show_name no)
